File: Schematics/Möbius Feedbacker/Möbius Feedbacker.sch (KiCad schematic (older format))
At the start: 23 parts

Commit message: Add schematic pdfs, change name to Pathway, update README
Parts:
- gave numbers to parts that had none: 23
Connections:
- net Mixer Circuit/Output1 renamed Mixer Circuit T/Output1
- net Mixer Circuit/Output2 renamed Mixer Circuit T/Output2
