File: Schematics/Möbius Feedbacker/VCACircuit.sch (KiCad schematic (older format))
At the start: 22 parts

Commit message: Add schematic pdfs, change name to Pathway, update README
Parts:
- gave numbers to parts that had none: 20
